File: PTP_Dario_Ladovic_project1/PTP_Dario_Ladovic_project1.kicad_sch (KiCad schematic)
At the start: 24 parts, among them U1 NE555P, U2 LM2574N-5

Commit message: LV3
Parts:
- removed R3: 2k, symbol Device:R_Small
- added R7: 10K, symbol Device:R_Small
- added U3: ~, SOT_23_6:DIP-6_102_ELL, symbol SN74LVC1G11:SN74LVC1G11
- renumbered C4 to C1, C5 to C2, D2 to D1, D3 to D2, D4 to D3, D5 to D4, D1 to D4, R5 to R1, R4 to R13, R6 to R2, R7 to R3, R8 to R4, U2 to U1
Connections:
- net +5V: now also R7.1, U3.5 (VCC)
- net Clock: now also R7.2
- net GND: now also U3.2 (GND)
- net Q1: now also U3.1 (A)
- net Q3: now also U3.3 (B)
- new net CLOCK: U3.6 (C)
- new net RESET: U3.4 (Y)
Other:
- moved on the sheet: SW2

Commit message: Vjezba 6. tjedan
Parts:
- added H1, H2, H3, H4: MountingHole, symbol Mechanical:MountingHole
- added R10, R11, R12, R15, R9: 10k, symbol Device:R_Small
- added R14, R17, R18, R5, R6, R8: 2k, symbol Device:R_Small
- added U2, U4: 4027, symbol 4xxx:4027
- added unit 3 of U3
- added U4: 74LS47, symbol 74xx:74LS47
- added U5: FYS-3911BUHR-21, Display_7Segment:HDSP-A151, symbol Display_Character:HDSP-7501
- C1: footprint (none) -> Capacitor_THT:CP_Radial_D5.0mm_P2.00mm; Manufacturer (none) -> AISHI; Manufacturer Part Number (none) -> EWH1EM220D11OT
- C2: footprint (none) -> Capacitor_THT:CP_Radial_D5.0mm_P2.00mm; Manufacturer (none) -> SAMWHA; Manufacturer Part Number (none) -> RD1A227M05011BB
Connections:
- net +5V: now also R10.1, R11.1, R12.1, R15.1, R9.1, U2.16 (VDD), U3.16 (VDD), U5.1 (CA), U5.6 (CA)
- net GND: now also C3.2, R13.2, SW2.3 (A), U2.7 (S), U2.8 (VSS), U2.9 (S), U3.8 (VSS), U4.7 (S), U4.8 (GND), U4.9 (S)
- net Q0: now also U2.13 (C), U4.1 (Q), U4.7 (A)
- net Q1: now also U2.15 (Q), U2.3 (C), U4.1 (B)
- net Q2: now also U2.1 (Q), U4.13 (C), U4.2 (C)
- net Q3: now also U4.15 (Q), U4.6 (D)
- new net: R10.2, U2.10 (J), U2.11 (K)
- new net: R14.1, U4.10 (d)
- new net: R8.1, U4.11 (c)
- new net: R6.1, U4.12 (b)
- new net: R5.1, U4.13 (a)
- new net: R18.1, U4.14 (g)
- new net: R17.1, U4.15 (f)
- new net: R15.2, U4.3 (LT), U4.4 (BI), U4.5 (RBI)
- new net: R8.1, U4.9 (e)
- new net: R6.2, U5.9 (B)
- new net: R12.2, U4.10 (J), U4.11 (K)
- new net: R9.2, U4.5 (K), U4.6 (J)
- new net: R5.2, U5.10 (A)
- new net: R18.2, U5.3 (G)
- new net: R11.2, U2.5 (K), U2.6 (J)
- new net: R17.2, U5.2 (F)
- new net: R8.2, U5.4 (E)
- new net: R14.2, U5.5 (D)
- new net: R8.2, U5.8 (C)
- new net Reset: U2.12 (R), U2.4 (R), U4.12 (R), U4.4 (R)
- new net clock: U4.3 (C)
- no-connect marks 1 -> 6
Other:
- moved on the sheet: C1, C2, C3, D1, D2, D3, D4, R1, R13, R2, R3, R4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

Commit message: Promjena grešaka
Parts:
- removed unit 3 of U3
- removed unit 2 of U4
- added U6: 4027, symbol 4xxx:4027
- renumbered C2 to C4, C1 to C5, D4 to D5, R1 to R19, R2 to R20, U1 to U7
Connections:
- net +5V: now also U6.16 (VDD)
- net Clock: now also U2.3 (C)
- net GND: now also U2.12 (R), U2.4 (R), U6.12 (R), U6.4 (R), U6.8 (VSS); no longer U2.7 (S), U2.9 (S)
- net Q0: now also U2.2 (~{Q})
- net Q1: now also U2.14 (~{Q}), U6.3 (C); no longer U2.15 (Q), U2.3 (C)
- net Q2: now also U6.13 (C), U6.2 (~{Q}); no longer U2.1 (Q)
- net Q3: now also U6.14 (~{Q})
- net Reset: now also U2.7 (S), U2.9 (S), U6.7 (S), U6.9 (S); no longer U2.12 (R), U2.4 (R)
- net at R12.2: now also U6.10 (J), U6.11 (K)
- net at R9.2: now also U2.5 (K), U2.6 (J)
- new net: R11.2, U6.5 (K), U6.6 (J)

Commit message: Slaganje plocice za spajanje komponenata
Parts:
- added R8: 2k, Resistor_SMD:R_1206_3216Metric_Pad1.30x1.75mm_HandSolder, symbol Device:R_Small
- C3, C4, C5: footprint (none) -> Capacitor_SMD:C_1206_3216Metric_Pad1.33x1.80mm_HandSolder
- D1, D2, D3, D5: footprint (none) -> LED_THT:LED_D5.0mm
- D4: footprint (none) -> Diode_THT:D_DO-41_SOD81_P12.70mm_Horizontal
- H1, H2, H3, H4: footprint (none) -> MountingHole:MountingHole_5.5mm
- J1: footprint (none) -> TerminalBlock_MetzConnect:TerminalBlock_MetzConnect_Type011_RT05502HBLC_1x02_P5.00mm_Horizontal
- L1: footprint (none) -> Inductor_THT:L_Radial_D7.2mm_P3.00mm_Murata_1700
- R1, R2, R3, R4: footprint (none) -> Resistor_THT:R_Axial_DIN0207_L6.3mm_D2.5mm_P10.16mm_Horizontal
- R10, R11, R12, R13, R14, R15, R17, R18, R19, R20, R5, R6, R7, R9: footprint (none) -> Resistor_SMD:R_1206_3216Metric_Pad1.30x1.75mm_HandSolder
- R16: renamed from R8; footprint (none) -> Resistor_SMD:R_1206_3216Metric_Pad1.30x1.75mm_HandSolder
- SW1: footprint (none) -> Button_Switch_THT:SW_PUSH_6mm_H4.3mm
- SW2: footprint Button_Switch_SMD:Nidec_Copal_CAS-120A -> Button_Switch_THT:SW_Slide_SPDT_Straight_CK_OS102011MS2Q
- U2, U4: footprint (none) -> Package_DIP:DIP-16_W7.62mm_Socket_LongPads
- U3: renamed from U6; footprint (none) -> Package_DIP:DIP-16_W7.62mm_Socket_LongPads
- U5: footprint Display_7Segment:HDSP-A151 -> Display_7Segment:HDSP-7401
- U6: renamed from U3; footprint SOT_23_6:DIP-6_102_ELL -> Package_TO_SOT_SMD:SOT-23-6
Connections:
- net GND: no longer C3.2, R13.2, SW2.3 (A)
- net at U4.11 (c): now also R8.1; no longer R16.1
- net at U5.8 (C): now also R8.2; no longer R16.2
- new net: C3.2, R13.2, SW2.3 (A)
Changed lines of the file:
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@@
 	)
 	(junction
-		(at 38.1 87.63)
-		(diameter 0)
-		(color 0 0 0 0)
-	)
-	(junction
 		(at 217.17 110.49)
 		(diameter 0)
@@
 	)
 	(junction
-		(at 30.48 87.63)
-		(diameter 0)
-		(color 0 0 0 0)
-	)
-	(junction
 		(at 217.17 113.03)
 		(diameter 0)
@@
 	(wire
 		(pts
-			(xy 38.1 87.63) (xy 30.48 87.63)
-		)
-		(stroke
-			(width 0)
-			(type default)
-		)
-	)
-	(wire
-		(pts
 			(xy 217.17 95.25) (xy 220.98 95.25)
 		)
@@
 			)
 		)
-		(property "Footprint" ""
+		(property "Footprint" "MountingHole:MountingHole_5.5mm"
 			(at 212.09 158.75 0)
 			(effects
@@
 			)
 		)
-		(property "Footprint" ""
+		(property "Footprint" "MountingHole:MountingHole_5.5mm"
 			(at 212.09 139.7 0)
 			(effects
@@
 			)
 		)
-		(property "Footprint" ""
+		(property "Footprint" "Package_DIP:DIP-16_W7.62mm_Socket_LongPads"
 			(at 102.87 107.95 0)
 			(effects
@@
 			)
 		)
-		(property "Footprint" ""
+		(property "Footprint" "Package_DIP:DIP-16_W7.62mm_Socket_LongPads"
 			(at 233.68 102.87 0)
 			(effects
@@
 		(dnp no)
 		(fields_autoplaced yes)
-		(property "Reference" "U6"
+		(property "Reference" "U3"
 			(at 158.3533 97.79 0)
 			(effects
@@
 			)
 		)
-		(property "Footprint" ""
+		(property "Footprint" "Package_DIP:DIP-16_W7.62mm_Socket_LongPads"
 			(at 156.21 107.95 0)
 			(effects
@@
 			(project ""
 				(path "/70e458e7-9e42-4bc9-991d-1fa23104cdd7"
-					(reference "U6")
+					(reference "U3")
 					(unit 1)
 				)
@@
 			)
 		)
-		(property "Footprint" ""
+		(property "Footprint" "Resistor_SMD:R_1206_3216Metric_Pad1.30x1.75mm_HandSolder"
 			(at 38.1 100.33 0)
 			(effects
@@
 			)
 		)
-		(property "Footprint" ""
+		(property "Footprint" "Resistor_THT:R_Axial_DIN0207_L6.3mm_D2.5mm_P10.16mm_Horizontal"
 			(at 256.54 55.118 90)
 			(effects
@@
 			)
 		)
-		(property "Footprint" ""
+		(property "Footprint" "Resistor_SMD:R_1206_3216Metric_Pad1.30x1.75mm_HandSolder"
 			(at 255.27 91.44 0)
 			(effects
@@
 			)
 		)
-		(property "Footprint" ""
+		(property "Footprint" "Resistor_THT:R_Axial_DIN0207_L6.3mm_D2.5mm_P10.16mm_Horizontal"
 			(at 256.54 32.258 90)
 			(effects
@@
 			)
 		)
-		(property "Footprint" ""
+		(property "Footprint" "Resistor_SMD:R_1206_3216Metric_Pad1.30x1.75mm_HandSolder"
 			(at 88.9 99.06 0)
 			(effects
@@
 		(dnp no)
 		(fields_autoplaced yes)
-		(property "Reference" "U6"
+		(property "Reference" "U3"
 			(at 191.77 38.0999 0)
 			(effects
@@
 			)
 		)
-		(property "Footprint" ""
+		(property "Footprint" "Package_DIP:DIP-16_W7.62mm_Socket_LongPads"
 			(at 185.42 39.37 0)
 			(effects
@@
 			(project ""
 				(path "/70e458e7-9e42-4bc9-991d-1fa23104cdd7"
-					(reference "U6")
+					(reference "U3")
 					(unit 3)
 				)
@@
 			)
 		)
-		(property "Footprint" ""
+		(property "Footprint" "LED_THT:LED_D5.0mm"
 			(at 242.57 38.1 0)
 			(effects
@@
 			)
 		)
-		(property "Footprint" ""
+		(property "Footprint" "Resistor_SMD:R_1206_3216Metric_Pad1.30x1.75mm_HandSolder"
 			(at 255.27 86.36 0)
 			(effects
@@
 			)
 		)
-		(property "Footprint" ""
+		(property "Footprint" "Resistor_SMD:R_1206_3216Metric_Pad1.30x1.75mm_HandSolder"
 			(at 255.27 118.11 0)
 			(effects
@@
 			)
 		)
-		(property "Footprint" ""
+		(property "Footprint" "LED_THT:LED_D5.0mm"
 			(at 242.57 53.34 0)
 			(effects
@@
 		(dnp no)
 		(fields_autoplaced yes)
-		(property "Reference" "U3"
+		(property "Reference" "U6"
 			(at 147.32 165.0298 0)
 			(effects
@@
 			)
 		)
-		(property "Footprint" "SOT_23_6:DIP-6_102_ELL"
+		(property "Footprint" "Package_TO_SOT_SMD:SOT-23-6"
 			(at 152.4 163.83 0)
 			(effects
@@
 			(project ""
 				(path "/70e458e7-9e42-4bc9-991d-1fa23104cdd7"
-					(reference "U3")
+					(reference "U6")
 					(unit 1)
 				)
@@
 			)
 		)
-		(property "Footprint" ""
+		(property "Footprint" "Capacitor_SMD:C_1206_3216Metric_Pad1.33x1.80mm_HandSolder"
 			(at 19.05 179.07 0)
 			(effects
@@
 			)
 		)
-		(property "Footprint" ""
+		(property "Footprint" "LED_THT:LED_D5.0mm"
 			(at 242.57 30.48 0)
 			(effects
@@
 			)
 		)
-		(property "Footprint" ""
+		(property "Footprint" "Capacitor_SMD:C_1206_3216Metric_Pad1.33x1.80mm_HandSolder"
 			(at 38.1 86.6648 0)
 			(effects
@@
 			)
 		)
-		(property "Footprint" ""
+		(property "Footprint" "Resistor_SMD:R_1206_3216Metric_Pad1.30x1.75mm_HandSolder"
 			(at 209.55 107.95 0)
 			(effects
@@
 			)
 		)
-		(property "Footprint" ""
+		(property "Footprint" "Package_DIP:DIP-16_W7.62mm_Socket_LongPads"
 			(at 153.67 39.37 0)
 			(effects
@@
 			)
 		)
-		(property "Footprint" ""
+		(property "Footprint" "Capacitor_SMD:C_1206_3216Metric_Pad1.33x1.80mm_HandSolder"
 			(at 35.56 152.4 0)
 			(effects
@@
 			)
 		)
-		(property "Footprint" ""
+		(property "Footprint" "Resistor_SMD:R_1206_3216Metric_Pad1.30x1.75mm_HandSolder"
 			(at 19.05 149.86 0)
 			(effects
@@
 			)
 		)
-		(property "Footprint" ""
+		(property "Footprint" "LED_THT:LED_D5.0mm"
 			(at 242.57 45.72 0)
 			(effects
@@
 			)
 		)
-		(property "Footprint" ""
+		(property "Footprint" "Button_Switch_THT:SW_PUSH_6mm_H4.3mm"
 			(at 29.21 95.25 0)
 			(effects
@@
 			)
 		)
-		(property "Footprint" ""
+		(property "Footprint" "Resistor_SMD:R_1206_3216Metric_Pad1.30x1.75mm_HandSolder"
 			(at 146.05 97.79 0)
 			(effects
@@
 			)
 		)
-		(property "Footprint" "Display_7Segment:HDSP-A151"
+		(property "Footprint" "Display_7Segment:HDSP-7401"
 			(at 273.05 116.84 0)
 			(effects
@@
 			)
 		)
-		(property "Footprint" ""
+		(property "Footprint" "Resistor_THT:R_Axial_DIN0207_L6.3mm_D2.5mm_P10.16mm_Horizontal"
 			(at 256.54 36.322 90)
 			(effects
@@
 			)
 		)
-		(property "Footprint" ""
+		(property "Footprint" "Package_DIP:DIP-16_W7.62mm_Socket_LongPads"
 			(at 128.27 107.95 0)
 			(effects
@@
 			)
 		)
-		(property "Footprint" ""
+		(property "Footprint" "TerminalBlock_MetzConnect:TerminalBlock_MetzConnect_Type011_RT05502HBLC_1x02_P5.00mm_Horizontal"
 			(at 24.13 35.56 0)
 			(effects
@@
 		(dnp no)
 		(fields_autoplaced yes)
-		(property "Reference" "U6"
+		(property "Reference" "U3"
 			(at 185.0233 97.79 0)
 			(effects
@@
 			)
 		)
-		(property "Footprint" ""
+		(property "Footprint" "Package_DIP:DIP-16_W7.62mm_Socket_LongPads"
 			(at 182.88 107.95 0)
 			(effects
@@
 			(project ""
 				(path "/70e458e7-9e42-4bc9-991d-1fa23104cdd7"
-					(reference "U6")
+					(reference "U3")
 					(unit 2)
 				)
@@
 			)
 		)
-		(property "Footprint" ""
+		(property "Footprint" "Resistor_SMD:R_1206_3216Metric_Pad1.30x1.75mm_HandSolder"
 			(at 255.27 113.03 0)
 			(effects
@@
 			)
 		)
-		(property "Footprint" ""
+		(property "Footprint" "Resistor_SMD:R_1206_3216Metric_Pad1.30x1.75mm_HandSolder"
 			(at 255.27 107.95 0)
 			(effects
@@
 			)
 		)
-		(property "Footprint" ""
+		(property "Footprint" "Resistor_SMD:R_1206_3216Metric_Pad1.30x1.75mm_HandSolder"
 			(at 255.27 96.52 0)
 			(effects
@@
 			)
 		)
-		(property "Footprint" ""
+		(property "Footprint" "MountingHole:MountingHole_5.5mm"
 			(at 212.09 146.05 0)
 			(effects
@@
 			)
 		)
-		(property "Footprint" "Button_Switch_SMD:Nidec_Copal_CAS-120A"
+		(property "Footprint" "Button_Switch_THT:SW_Slide_SPDT_Straight_CK_OS102011MS2Q"
 			(at 53.34 113.03 0)
 			(effects
@@
 			)
 		)
-		(property "Footprint" ""
+		(property "Footprint" "Inductor_THT:L_Radial_D7.2mm_P3.00mm_Murata_1700"
 			(at 104.14 35.56 0)
 			(effects
@@
 			)
 		)
-		(property "Footprint" ""
+		(property "Footprint" "Resistor_SMD:R_1206_3216Metric_Pad1.30x1.75mm_HandSolder"
 			(at 170.18 97.79 0)
 			(effects
@@
 			)
 		)
-		(property "Footprint" ""
+		(property "Footprint" "Resistor_SMD:R_1206_3216Metric_Pad1.30x1.75mm_HandSolder"
 			(at 118.11 99.06 0)
 			(effects
@@
 			)
 		)
-		(property "Footprint" ""
+		(property "Footprint" "Diode_THT:D_DO-41_SOD81_P12.70mm_Horizontal"
 			(at 96.52 48.26 0)
 			(effects
@@
 			)
 		)
-		(property "Footprint" ""
+		(property "Footprint" "Resistor_SMD:R_1206_3216Metric_Pad1.30x1.75mm_HandSolder"
 			(at 19.05 161.29 0)
 			(effects
@@
 			)
 		)
-		(property "Footprint" ""
+		(property "Footprint" "Resistor_SMD:R_1206_3216Metric_Pad1.30x1.75mm_HandSolder"
 			(at 255.27 102.87 0)
 			(effects
@@
 			)
 		)
-		(property "Footprint" ""
+		(property "Footprint" "Resistor_THT:R_Axial_DIN0207_L6.3mm_D2.5mm_P10.16mm_Horizontal"
 			(at 256.54 47.498 90)
 			(effects
@@
 			)
 		)
-		(property "Footprint" ""
+		(property "Footprint" "MountingHole:MountingHole_5.5mm"
 			(at 212.09 152.4 0)
 			(effects
@@
 			)
 		)
-		(property "Footprint" ""
+		(property "Footprint" "Resistor_SMD:R_1206_3216Metric_Pad1.30x1.75mm_HandSolder"
 			(at 60.96 95.25 0)
 			(effects
