File: PTP_Dario_Ladovic_project1/PTP_Dario_Ladovic_project1.kicad_pcb (KiCad board)
At the start: 2 copper layers, 100 x 80 mm, 45 parts, among them U1 LM2574N-5, U2 4027, U3 4027, U4 74LS47, U5 FYS-3911BUHR-21, U7 NE555P

Commit message: Dokumentiranje
Parts:
- moved U1 11.2 mm to (130.3, 65.8), turned to 180 degrees
- moved R1 10.2 mm to (176.0, 62.1), turned to 90 degrees
- moved R4 10.1 mm to (150.5, 62.1), turned to 90 degrees
- moved R3 10.0 mm to (159.0, 62.0), turned to 90 degrees
Routing:
- net GND: track 0.00 -> 317.6 mm, vias 0 -> 2
- net +5V: track 0.00 -> 245.7 mm, vias 0 -> 7
- net Q3: track 0.00 -> 71.5 mm, vias 0 -> 3
- net Q0: track 0.00 -> 64.2 mm, vias 0 -> 3
- net Q1: track 0.00 -> 54.7 mm
- net Clock: track 0.00 -> 41.2 mm, vias 0 -> 1
- net Q2: track 0.00 -> 34.5 mm, vias 0 -> 2
- net Net-(SW2-A): track 0.00 -> 32.9 mm
- net Reset: track 0.00 -> 30.4 mm, vias 0 -> 2
- net Net-(U5-B): track 0.00 -> 26.2 mm
- net 555: track 0.00 -> 25.7 mm
- net Net-(U2A-J): track 0.00 -> 24.1 mm, vias 0 -> 1
- net VD: track 0.00 -> 23.1 mm
- net Net-(D4-K): track 0.00 -> 23.0 mm
- net Net-(U4-BI): track 0.00 -> 22.9 mm
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